Commit message: adding contact sensor

File: src/singlebot_config/urdf/singlebot.urdf (robot description, URDF)
Before this commit: robot single_world, 5 links, 4 joints
Joints:
- joint foot_back_joint: limit lower=-0.1 upper=0.2 effort=20 velocity=1.0 -> lower=-0.3 upper=0.3 effort=20 velocity=1.0

Commit message: hopping

File: src/singlebot_config/urdf/singlebot.urdf (robot description, URDF)
Before this commit: robot single_world, 5 links, 4 joints
Links:
- link foot_back: geometry collision cylinder length=0.6 radius=0.05; collision sphere radius=0.05
- link leg_back: geometry collision cylinder length=0.6 radius=0.05; collision sphere radius=0.05
Joints:
- joint foot_back_joint: limit lower=-0.3 upper=0.3 effort=20 velocity=1.0 -> lower=-1.0 upper=1.0 effort=100 velocity=100.0; origin xyz=0 0 0.3 rpy=0 0 0 -> xyz=0 0 0.6 rpy=0 0 0
- joint hip_back_joint: origin xyz=0 0 -0.3 rpy=0 0 0 -> xyz=0 0 0 rpy=0 0 0

Commit message: slip final

File: src/singlebot_config/urdf/singlebot.urdf (robot description, URDF)
Before this commit: robot single_world, 5 links, 4 joints
Links:
- link robot_base: geometry collision sphere radius=0.3; visual sphere radius=0.1
Joints:
- joint foot_back_joint: limit lower=-1.0 upper=1.0 effort=100 velocity=100.0 -> lower=-1.0 upper=1.0 effort=10000 velocity=100.0
- joint leg_back_joint: axis 0 1 0 -> 0 -1 0
