Commit message: modified model and figure

File: src/singlebot_config/urdf/trirot.urdf (robot description, URDF)
Before this commit: robot single_world, 13 links, 12 joints
Links:
- link leg_back: geometry visual cylinder length=0.6 radius=0.05; visual sphere radius=0.05
- link leg_left: geometry visual cylinder length=0.6 radius=0.05; visual sphere radius=0.05
- link leg_right: geometry visual cylinder length=0.6 radius=0.05; visual sphere radius=0.05
