Commit message: slip works 100

File: src/singlebot_config/urdf/singlerot.urdf (robot description, URDF)
Before this commit: robot single_world, 7 links, 6 joints
Links:
- link base1_link: geometry visual sphere radius=0.02
- link base2_link: geometry visual sphere radius=0.02
- link foot_back: geometry collision cylinder length=0.6 radius=0.02; collision sphere radius=0.02
- link hip_back: geometry collision sphere radius=0.02; visual sphere radius=0.02
- link leg_back: geometry collision cylinder length=0.3 radius=0.02; collision sphere radius=0.02
Joints:
- joint foot_back_joint: limit lower=-1.2 upper=1.2 effort=10000 velocity=150.0 -> lower=-1.0 upper=1.2 effort=1000 velocity=4
- joint hip_back_joint: limit (none) -> lower=-9 upper=9 effort=100 velocity=3.0
- joint leg_back_joint: limit (none) -> lower=-9 upper=9 effort=100 velocity=3.0

Commit message: make model prettier:

File: src/singlebot_config/urdf/singlerot.urdf (robot description, URDF)
Before this commit: robot single_world, 7 links, 6 joints
Links:
- link leg_back: geometry visual cylinder length=0.6 radius=0.05; visual sphere radius=0.05
